File: 3bit_ttl_calculator.sch (KiCad schematic (older format))
At the start: 135 parts, among them Q1 BC547, Q10 BC547, Q11 BC547, Q12 BC547, Q13 BC547, Q14 BC547, Q15 BC547, Q16 BC547, Q17 BC547, Q18 BC547, Q19 BC547, Q2 BC547, Q20 BC547, Q21 BC547, Q22 BC547, Q23 BC547, Q24 BC547, Q25 BC547, Q26 BC547, Q27 BC547, Q28 BC547, Q29 BC547, Q3 BC547, Q30 BC547, Q31 BC547, Q32 BC547, Q33 BC547, Q34 BC547, Q35 BC547, Q36 BC547, Q37 BC547, Q38 BC547, Q39 BC547, Q4 BC547, Q40 BC547, Q41 BC547, Q42 BC547, Q43 BC547, Q44 BC547, Q45 BC547, Q46 BC547, Q47 BC547, Q48 BC547, Q49 BC547, Q5 BC547, Q50 BC547, Q51 BC547, Q52 BC547, Q53 BC547, Q54 BC547, Q6 BC547, Q7 BC547, Q8 BC547, Q9 BC547

Commit message: fix labels. add input/output components
Parts:
- added D1, D2, D3, D4: LED, symbol Device:LED
- added J1, J2: Conn_01x03_Female, symbol Connector:Conn_01x03_Female
Connections:
- net A1: now also J1.1 (Pin_1)
- net A2: now also J1.2 (Pin_2); no longer R4.2, R5.2, R6.2
- net B1: now also J2.1 (Pin_1)
- net Cout3: now also D4.2 (A)
- net GND: now also D1.1 (K), D2.1 (K), D3.1 (K), D4.1 (K)
- net S1: now also D1.2 (A)
- net S2: now also D2.2 (A)
- net S3: now also D3.2 (A)
- new net A3: J1.3 (Pin_3), R5.2
- new net B2: J2.2 (Pin_2), R4.2
- new net B3: J2.3 (Pin_3), R6.2
Other:
- note added: "Input"
- note added: "Output"
Changed lines of the file:
@@
 A2
 Text GLabel 1300 13250 0    50   Input ~ 0
-A2
+A3
 Text GLabel 1300 8850 0    50   Input ~ 0
-A2
+B2
 Text GLabel 1300 13800 0    50   Input ~ 0
-A2
+B3
 Wire Wire Line
 	1300 8300 2000 8300
@@
 	6750 12350 6750 13050
 Connection ~ 6750 13050
+$Comp
+L Connector:Conn_01x03_Female J1
+U 1 1 5EDF6A0A
+P 13800 1500
+F 0 "J1" H 13828 1526 50  0000 L CNN
+F 1 "Conn_01x03_Female" H 13828 1435 50  0000 L CNN
+F 2 "" H 13800 1500 50  0001 C CNN
+F 3 "~" H 13800 1500 50  0001 C CNN
+	1    13800 1500
+	1    0    0    -1
+$EndComp
+$Comp
+L Connector:Conn_01x03_Female J2
+U 1 1 5EDF7BF3
+P 13800 1900
+F 0 "J2" H 13828 1926 50  0000 L CNN
+F 1 "Conn_01x03_Female" H 13828 1835 50  0000 L CNN
+F 2 "" H 13800 1900 50  0001 C CNN
+F 3 "~" H 13800 1900 50  0001 C CNN
+	1    13800 1900
+	1    0    0    -1
+$EndComp
+$Comp
+L Device:LED D1
+U 1 1 5EDF85E5
+P 15800 1750
+F 0 "D1" V 15839 1633 50  0000 R CNN
+F 1 "LED" V 15748 1633 50  0000 R CNN
+F 2 "" H 15800 1750 50  0001 C CNN
+F 3 "~" H 15800 1750 50  0001 C CNN
+	1    15800 1750
+	0    -1   -1   0
+$EndComp
+$Comp
+L Device:LED D2
+U 1 1 5EDF966B
+P 16100 1750
+F 0 "D2" V 16139 1633 50  0000 R CNN
+F 1 "LED" V 16048 1633 50  0000 R CNN
+F 2 "" H 16100 1750 50  0001 C CNN
+F 3 "~" H 16100 1750 50  0001 C CNN
+	1    16100 1750
+	0    -1   -1   0
+$EndComp
+$Comp
+L Device:LED D3
+U 1 1 5EDF9B28
+P 16400 1750
+F 0 "D3" V 16439 1633 50  0000 R CNN
+F 1 "LED" V 16348 1633 50  0000 R CNN
+F 2 "" H 16400 1750 50  0001 C CNN
+F 3 "~" H 16400 1750 50  0001 C CNN
+	1    16400 1750
+	0    -1   -1   0
+$EndComp
+$Comp
+L Device:LED D4
+U 1 1 5EDF9FE6
+P 16650 1750
+F 0 "D4" V 16689 1633 50  0000 R CNN
+F 1 "LED" V 16598 1633 50  0000 R CNN
+F 2 "" H 16650 1750 50  0001 C CNN
+F 3 "~" H 16650 1750 50  0001 C CNN
+	1    16650 1750
+	0    -1   -1   0
+$EndComp
+Text GLabel 15800 1500 1    50   Input ~ 0
+S1
+Wire Wire Line
+	15800 1500 15800 1600
+Text GLabel 16100 1500 1    50   Input ~ 0
+S2
+Text GLabel 16400 1500 1    50   Input ~ 0
+S3
+Wire Wire Line
+	16400 1500 16400 1600
+Wire Wire Line
+	16100 1500 16100 1600
+Text GLabel 16650 1500 1    50   Input ~ 0
+Cout3
+Wire Wire Line
+	16650 1500 16650 1600
+Text GLabel 15800 2100 3    50   Input ~ 0
+GND
+Wire Wire Line
+	15800 2100 15800 2000
+Wire Wire Line
+	15800 2000 16100 2000
+Wire Wire Line
+	16100 2000 16100 1900
+Connection ~ 15800 2000
+Wire Wire Line
+	15800 2000 15800 1900
+Wire Wire Line
+	16100 2000 16400 2000
+Wire Wire Line
+	16400 2000 16400 1900
+Connection ~ 16100 2000
+Wire Wire Line
+	16400 2000 16650 2000
+Wire Wire Line
+	16650 2000 16650 1900
+Connection ~ 16400 2000
+Text GLabel 13500 1400 0    50   Input ~ 0
+A1
+Text GLabel 13500 1500 0    50   Input ~ 0
+A2
+Text GLabel 13500 1600 0    50   Input ~ 0
+A3
+Text GLabel 13500 1800 0    50   Input ~ 0
+B1
+Text GLabel 13500 1900 0    50   Input ~ 0
+B2
+Text GLabel 13500 2000 0    50   Input ~ 0
+B3
+Wire Wire Line
+	13500 1400 13600 1400
+Wire Wire Line
+	13500 1500 13600 1500
+Wire Wire Line
+	13500 1600 13600 1600
+Wire Wire Line
+	13500 1800 13600 1800
+Wire Wire Line
+	13500 1900 13600 1900
+Wire Wire Line
+	13500 2000 13600 2000
+Wire Notes Line
+	13000 1000 13000 2200
+Wire Notes Line
+	13000 2200 14700 2200
+Wire Notes Line
+	14700 2200 14700 1000
+Wire Notes Line
+	14700 1000 13000 1000
+Wire Notes Line
+	15150 2400 17100 2400
+Wire Notes Line
+	17100 2400 17100 1000
+Wire Notes Line
+	17100 1000 15150 1000
+Wire Notes Line
+	15150 1000 15150 2400
+Text Notes 15200 1100 0    50   ~ 0
+Output
+Text Notes 13050 1100 0    50   ~ 0
+Input
 $EndSCHEMATC

Commit message: fix schematics, add board design...
Parts:
- added J3: Conn_01x02_Female, Connector_PinHeader_2.54mm:PinHeader_1x02_P2.54mm_Vertical, symbol Connector:Conn_01x02_Female
- D1, D2, D3, D4: footprint (none) -> LED_THT:LED_D3.0mm
- J1, J2: footprint (none) -> Connector_PinHeader_2.54mm:PinHeader_1x03_P2.54mm_Vertical
- R1, R10, R11, R12, R13, R14, R15, R16, R17, R18, R19, R2, R20, R21, R22, R23, R24, R25, R26, R27, R28, R29, R3, R30, R31, R32, R33, R34, R35, R36, R37, R38, R39, R4, R40, R41, R42, R43, R44, R45, R46, R47, R48, R49, R5, R50, R51, R52, R53, R54, R55, R56, R57, R58, R59, R6, R60, R61, R62, R63, R64, R65, R66, R67, R68, R69, R7, R70, R71, R72, R73, R74, R75, R76, R77, R78, R79, R8, R80, R81, R9: footprint (none) -> Resistor_THT:R_Axial_DIN0207_L6.3mm_D2.5mm_P10.16mm_Horizontal
Connections:
- net A1: no longer R14.2, R18.2
- net A2: now also R14.2
- net A3: now also R18.2
- net B1: no longer R17.2, R21.2
- net B2: now also R17.2
- net B3: now also R21.2
- net GND: now also J3.2 (Pin_2)
- net Vcc: now also J3.1 (Pin_1)
